File: kicad/koziol_drone_v1/BMP388.kicad_sch (KiCad schematic)
At the start: 3 parts, among them U4 BMP388

Commit message: scheme descriptions and PDF plot
Other:
- note added: "BMP388"
- note added: "Barometer"
Changed lines of the file:
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@@
+		)
+	)
+	(text "Barometer"
+		(exclude_from_sim no)
+		(at 91.186 107.442 0)
+		(effects
+			(font
+				(size 2.54 2.54)
+			)
+			(justify left)
+		)
+	)
+	(text "BMP388"
+		(exclude_from_sim no)
+		(at 99.06 127.762 0)
+		(effects
+			(font
+				(size 2.54 2.54)
+			)
+			(justify left)
 		)
 	)
