File: kicad/koziol_drone_v1/HMC5883L.kicad_sch (KiCad schematic)
At the start: 5 parts, among them U3 HMC5883L

Commit message: scheme descriptions and PDF plot
Other:
- note added: "HMC588L"
- note added: "Magnetometer NEEDED LOW CAPACITOR ESR C5 I C6 (<200 OHM)"
- note removed: "WYMAGANY NISKI ESR KONDENSATOROW C5 I C6 (<200 OHM)"
Changed lines of the file:
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@@
 		)
 	)
-	(text "WYMAGANY NISKI ESR KONDENSATOROW C5 I C6 (<200 OHM)"
+	(text "Magnetometer\n\nNEEDED LOW CAPACITOR ESR C5 I C6 (<200 OHM)"
 		(exclude_from_sim no)
-		(at 101.346 88.646 0)
+		(at 90.932 112.014 0)
 		(effects
 			(font
-				(size 1.27 1.27)
+				(size 2.54 2.54)
+			)
+			(justify left)
+		)
+	)
+	(text "HMC588L"
+		(exclude_from_sim no)
+		(at 107.696 127.762 0)
+		(effects
+			(font
+				(size 2.54 2.54)
 			)
 		)
