File: kicad/koziol_drone_v1/MPU6050.kicad_sch (KiCad schematic)
At the start: 6 parts, among them U2 MPU-6050

Commit message: scheme descriptions and PDF plot
Other:
- note added: "Accelerometer and gyroscope"
- note added: "MPU6050"
Changed lines of the file:
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@@
+		)
+	)
+	(text "Accelerometer and gyroscope"
+		(exclude_from_sim no)
+		(at 119.634 107.696 0)
+		(effects
+			(font
+				(size 2.54 2.54)
+			)
+		)
+	)
+	(text "MPU6050"
+		(exclude_from_sim no)
+		(at 108.458 128.016 0)
+		(effects
+			(font
+				(size 2.54 2.54)
+			)
 		)
 	)
